File: hardware/archive/finn_recent/BREAD_Slice.kicad_pcb (KiCad board)
At the start: 2 copper layers, 70 x 100 mm, 48 parts, among them J1 Conn_01x10_Female, J10 Term_PressFit_Phoenix_Contact, J11 Term_PressFit_Phoenix_Contact, J12 Term_PressFit_Phoenix_Contact, J13 Term_PressFit_Phoenix_Contact, J14 Term_PressFit_Phoenix_Contact, J15 Term_PressFit_Phoenix_Contact, J16 Term_PressFit_Phoenix_Contact, J17 Term_PressFit_Phoenix_Contact, J18 Term_PressFit_Phoenix_Contact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

Commit message: added historical scripts and new revisions
Connections:
- net /CLK renamed /TC_CLK
- net /DATA renamed /TC_DATA
- net /I2C_CLK renamed /I2C_TC_CLK
Changed lines of the file:
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@@
 	(net 5 "+5V")
 	(net 6 "/LED")
-	(net 7 "/I2C_CLK")
+	(net 7 "/I2C_TC_CLK")
 	(net 8 "unconnected-(A1-D8-Pad11)")
 	(net 9 "/I2C_DAT")
@@
 	(net 20 "+12V")
 	(net 21 "/INT")
-	(net 22 "/DATA")
-	(net 23 "/CLK")
+	(net 22 "/TC_DATA")
+	(net 23 "/TC_CLK")
 	(net 24 "/SS1")
 	(net 25 "/SS2")
@@
 			)
 		)
-		(property "Datasheet" ""
+		(property "TC_DATAsheet" ""
 			(at 0 0 0)
 			(unlocked yes)
@@
 			)
 		)
-		(property "Datasheet" ""
+		(property "TC_DATAsheet" ""
 			(at 0 0 0)
 			(unlocked yes)
@@
 			)
 		)
-		(property "Datasheet" ""
+		(property "TC_DATAsheet" ""
 			(at 0 0 0)
 			(unlocked yes)
@@
 			)
 		)
-		(property "Datasheet" ""
+		(property "TC_DATAsheet" ""
 			(at 0 0 0)
 			(unlocked yes)
@@
 			)
 		)
-		(property "Datasheet" ""
+		(property "TC_DATAsheet" ""
 			(at 0 0 0)
 			(unlocked yes)
@@
 			(layers "*.Cu" "*.Mask")
 			(remove_unused_layers no)
-			(net 22 "/DATA")
+			(net 22 "/TC_DATA")
 			(pinfunction "D12")
 			(pintype "bidirectional")
@@
 			(layers "*.Cu" "*.Mask")
 			(remove_unused_layers no)
-			(net 23 "/CLK")
+			(net 23 "/TC_CLK")
 			(pinfunction "D13")
 			(pintype "bidirectional")
@@
 			(layers "*.Cu" "*.Mask")
 			(remove_unused_layers no)
-			(net 7 "/I2C_CLK")
+			(net 7 "/I2C_TC_CLK")
 			(pinfunction "A5")
 			(pintype "bidirectional")
@@
 			)
 		)
-		(property "Datasheet" ""
+		(property "TC_DATAsheet" ""
 			(at 0 0 0)
 			(unlocked yes)
@@
 			(layers "*.Cu" "*.Mask")
 			(remove_unused_layers no)
-			(net 7 "/I2C_CLK")
+			(net 7 "/I2C_TC_CLK")
 			(pinfunction "Pin_3")
 			(pintype "passive")
@@
 			)
 		)
-		(property "Datasheet" ""
+		(property "TC_DATAsheet" ""
 			(at 0 0 -90)
 			(unlocked yes)
@@
 			)
 		)
-		(property "Datasheet" ""
+		(property "TC_DATAsheet" ""
 			(at 0 0 0)
 			(unlocked yes)
@@
 			)
 		)
-		(property "Datasheet" ""
+		(property "TC_DATAsheet" ""
 			(at 0 0 0)
 			(unlocked yes)
@@
 			)
 		)
-		(property "Datasheet" ""
+		(property "TC_DATAsheet" ""
 			(at 0 0 -90)
 			(unlocked yes)
@@
 			)
 		)
-		(property "Datasheet" ""
+		(property "TC_DATAsheet" ""
 			(at 0 0 0)
 			(unlocked yes)
@@
 			)
 		)
-		(property "Datasheet" ""
+		(property "TC_DATAsheet" ""
 			(at 0 0 0)
 			(unlocked yes)
@@
 			)
 		)
-		(property "Datasheet" ""
+		(property "TC_DATAsheet" ""
 			(at 0 0 0)
 			(unlocked yes)
@@
 			)
 		)
-		(property "Datasheet" ""
+		(property "TC_DATAsheet" ""
 			(at 0 0 0)
 			(unlocked yes)
@@
 			)
 		)
-		(property "Datasheet" ""
+		(property "TC_DATAsheet" ""
 			(at 0 0 0)
 			(unlocked yes)
@@
 			)
 		)
-		(property "Datasheet" ""
+		(property "TC_DATAsheet" ""
 			(at 0 0 0)
 			(unlocked yes)
@@
 			)
 		)
-		(property "Datasheet" ""
+		(property "TC_DATAsheet" ""
 			(at 0 0 0)
 			(unlocked yes)
@@
 			)
 		)
-		(property "Datasheet" ""
+		(property "TC_DATAsheet" ""
 			(at 0 0 0)
 			(unlocked yes)
@@
 			)
 		)
-		(property "Datasheet" ""
+		(property "TC_DATAsheet" ""
 			(at 0 0 0)
 			(unlocked yes)
@@
 			)
 		)
-		(property "Datasheet" ""
+		(property "TC_DATAsheet" ""
 			(at 0 0 0)
 			(unlocked yes)
@@
 			)
 		)
-		(property "Datasheet" ""
+		(property "TC_DATAsheet" ""
 			(at 0 0 0)
 			(unlocked yes)
@@
 			)
 		)
-		(property "Datasheet" ""
+		(property "TC_DATAsheet" ""
 			(at 0 0 -90)
 			(unlocked yes)
@@
 			)
 		)
-		(property "Datasheet" ""
+		(property "TC_DATAsheet" ""
 			(at 0 0 0)
 			(unlocked yes)
@@
 		(layer "F.Cu")
 		(at 173.3 136.132769)
-		(descr "<h3>WS2812B</h3>\n\n<p>Specifications:\n<ul><li>Pin count: 4</li>\n<li>Size: 5.0 x 5.0 mm</li>\n</ul></p>\n<p><b>Datasheet referenced for footprint:</b> <a href=\"http://cdn.sparkfun.com/datasheets/BreakoutBoards/WS2812B.pdf\">WS2812B</a></p>\n<p>Example device:\n<ul><li>WS2812B</li>")
+		(descr "<h3>WS2812B</h3>\n\n<p>Specifications:\n<ul><li>Pin count: 4</li>\n<li>Size: 5.0 x 5.0 mm</li>\n</ul></p>\n<p><b>TC_DATAsheet referenced for footprint:</b> <a href=\"http://cdn.sparkfun.com/TC_DATAsheets/BreakoutBoards/WS2812B.pdf\">WS2812B</a></p>\n<p>Example device:\n<ul><li>WS2812B</li>")
 		(property "Reference" "D1"
 			(at 0 0.6 0)
@@
 			)
 		)
-		(property "Datasheet" ""
+		(property "TC_DATAsheet" ""
 			(at 0 0 0)
 			(unlocked yes)
@@
 			)
 		)
-		(property "Datasheet" ""
+		(property "TC_DATAsheet" ""
 			(at 0 0 0)
 			(unlocked yes)
@@
 			)
 		)
-		(property "Datasheet" ""
+		(property "TC_DATAsheet" ""
 			(at 0 0 0)
 			(unlocked yes)
@@
 			)
 		)
-		(property "Datasheet" ""
+		(property "TC_DATAsheet" ""
 			(at 0 0 0)
 			(unlocked yes)
@@
 			)
 		)
-		(property "Datasheet" ""
+		(property "TC_DATAsheet" ""
 			(at 0 0 0)
 			(unlocked yes)
@@
 			)
 		)
-		(property "Datasheet" ""
+		(property "TC_DATAsheet" ""
 			(at 0 0 0)
 			(unlocked yes)
@@
 			)
 		)
-		(property "Datasheet" ""
+		(property "TC_DATAsheet" ""
 			(at 0 0 0)
 			(unlocked yes)
@@
 			)
 		)
-		(property "Datasheet" ""
+		(property "TC_DATAsheet" ""
 			(at 0 0 0)
 			(unlocked yes)
@@
 			)
 		)
-		(property "Datasheet" ""
+		(property "TC_DATAsheet" ""
 			(at 0 0 0)
 			(unlocked yes)
@@
 			)
 		)
-		(property "Datasheet" ""
+		(property "TC_DATAsheet" ""
 			(at 0 0 180)
 			(unlocked yes)
@@
 			(layers "B.Cu" "B.Paste" "B.Mask")
 			(roundrect_rratio 0.25)
-			(net 7 "/I2C_CLK")
+			(net 7 "/I2C_TC_CLK")
 			(pinfunction "Pin_4")
 			(pintype "passive")
@@
 			)
 		)
-		(property "Datasheet" ""
+		(property "TC_DATAsheet" ""
 			(at 0 0 90)
 			(unlocked yes)
@@
 			)
 		)
-		(property "Datasheet" ""
+		(property "TC_DATAsheet" ""
 			(at 0 0 0)
 			(unlocked yes)
@@
 			)
 		)
-		(property "Datasheet" ""
+		(property "TC_DATAsheet" ""
 			(at 0 0 180)
 			(unlocked yes)
@@
 			(layers "B.Cu" "B.Paste" "B.Mask")
 			(roundrect_rratio 0.07)
-			(net 23 "/CLK")
+			(net 23 "/TC_CLK")
 			(pinfunction "SCK")
 			(pintype "input")
@@
 			(layers "B.Cu" "B.Paste" "B.Mask")
 			(roundrect_rratio 0.07)
-			(net 22 "/DATA")
+			(net 22 "/TC_DATA")
 			(pinfunction "SO")
 			(pintype "output")
@@
 			)
 		)
-		(property "Datasheet" ""
+		(property "TC_DATAsheet" ""
 			(at 0 0 0)
 			(unlocked yes)
@@
 			)
 		)
-		(property "Datasheet" ""
+		(property "TC_DATAsheet" ""
 			(at 0 0 0)
 			(unlocked yes)
@@
 			)
 		)
-		(property "Datasheet" ""
+		(property "TC_DATAsheet" ""
 			(at 0 0 180)
 			(unlocked yes)
@@
 			)
 		)
-		(property "Datasheet" ""
+		(property "TC_DATAsheet" ""
 			(at 0 0 180)
 			(unlocked yes)
@@
 			)
 		)
-		(property "Datasheet" ""
+		(property "TC_DATAsheet" ""
 			(at 0 0 0)
 			(unlocked yes)
@@
 			)
 		)
-		(property "Datasheet" ""
+		(property "TC_DATAsheet" ""
 			(at 0 0 180)
 			(unlocked yes)
@@
 			)
 		)
-		(property "Datasheet" ""
+		(property "TC_DATAsheet" ""
 			(at 0 0 0)
 			(unlocked yes)
@@
 			)
 		)
-		(property "Datasheet" ""
+		(property "TC_DATAsheet" ""
 			(at 0 0 0)
 			(unlocked yes)
@@
 			)
 		)
-		(property "Datasheet" ""
+		(property "TC_DATAsheet" ""
 			(at 0 0 180)
 			(unlocked yes)
@@
 			)
 		)
-		(property "Datasheet" ""
+		(property "TC_DATAsheet" ""
 			(at 0 0 90)
 			(unlocked yes)
@@
 			)
 		)
-		(property "Datasheet" ""
+		(property "TC_DATAsheet" ""
 			(at 0 0 180)
 			(unlocked yes)
@@
 			(layers "B.Cu" "B.Paste" "B.Mask")
 			(roundrect_rratio 0.07)
-			(net 23 "/CLK")
+			(net 23 "/TC_CLK")
 			(pinfunction "SCK")
 			(pintype "input")
@@
 			(layers "B.Cu" "B.Paste" "B.Mask")
 			(roundrect_rratio 0.07)
-			(net 22 "/DATA")
+			(net 22 "/TC_DATA")
 			(pinfunction "SO")
 			(pintype "output")
@@
 			)
 		)
-		(property "Datasheet" ""
+		(property "TC_DATAsheet" ""
 			(at 0 0 0)
 			(unlocked yes)
