File: hardware/archive/finn_recent/BREAD_Slice.kicad_sch (KiCad schematic)
At the start: 47 parts, among them J1 Conn_01x10_Female, J10 Term_PressFit_Phoenix_Contact, J11 Term_PressFit_Phoenix_Contact, J12 Term_PressFit_Phoenix_Contact, J13 Term_PressFit_Phoenix_Contact, J14 Term_PressFit_Phoenix_Contact, J15 Term_PressFit_Phoenix_Contact, J16 Term_PressFit_Phoenix_Contact, J17 Term_PressFit_Phoenix_Contact, J18 Term_PressFit_Phoenix_Contact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

Commit message: added historical scripts and new revisions
Parts:
- A1: TC_DATAsheet (none) -> http://www.mouser.com/pdfdocs/Gravitech_Arduino_Nano3_0.pdf
- D1: TC_DATAsheet (none) -> https://cdn.sparkfun.com/TC_DATAsheets/BreakoutBoards/WS281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
- D2, D3: TC_DATAsheet (none) -> https://www.digikey.com/short/q75wqm
- F1, F2: TC_DATAsheet (none) -> https://www.digikey.com/short/q7wbwz
- J10, J11, J12, J13, J14, J15, J16, J17, J18, J3, J4, J5, J6, J7, J8, J9: TC_DATAsheet (none) -> https://mm.digikey.com/Volume0/opasTC_DATA/d220001/medias/d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
- K1, K2: TC_DATAsheet (none) -> https://www.omron.com/ecb/products/pdf/en-g5q.pdf
- U2, U5: TC_DATAsheet (none) -> http://www.vishay.com/docs/83510/tcmt1100.pdf
Connections:
- net CLK renamed TC_CLK
- net DATA renamed TC_DATA
- net I2C_CLK renamed I2C_TC_CLK
