File: hardware/archive/osf_2022-05-19/BREAD_Slice.kicad_sch (KiCad schematic)
At the start: 39 parts, among them J1 Conn_01x10_Female, J2 Term_2, J3 Term_2, J4 Term_2, J5 Term_2, J6 Term_2, J7 Term_2, J8 Term_2, K1 G5Q-1, Q1 TIP120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

Commit message: added historical scripts and new revisions
Parts:
- A1: TC_DATAsheet (none) -> http://www.mouser.com/pdfdocs/Gravitech_Arduino_Nano3_0.pdf
- C1, C2: TC_DATAsheet (none) -> https://www.digikey.com/short/qcd8n7
- D1, D2: TC_DATAsheet (none) -> https://www.digikey.com/short/q75wjm
- D3: TC_DATAsheet (none) -> https://www.digikey.com/short/q75wqm
- F1: TC_DATAsheet (none) -> https://www.digikey.com/short/q7wbwz
- J2, J3, J4, J5, J6, J7, J8: TC_DATAsheet (none) -> https://www.digikey.com/short/q7wbhd
- K1: TC_DATAsheet (none) -> https://www.omron.com/ecb/products/pdf/en-g5q.pdf
- Q1: TC_DATAsheet (none) -> https://www.onsemi.com/pub/Collateral/TIP120-D.PDF
- RV1, RV2: TC_DATAsheet (none) -> https://www.digikey.com/short/qt5j3q
- U1, U2: TC_DATAsheet (none) -> http://ww1.microchip.com/downloads/en/DeviceDoc/21733j.pdf
Connections:
- net CLK renamed TC_CLK
- net DATA renamed TC_DATA
- net I2C_CLK renamed I2C_TC_CLK
