File: hardware/archive/osf_2023-12-06/BREAD_Slice.kicad_pcb (KiCad board)
At the start: 2 copper layers, 70 x 100 mm, 38 parts, among them J1 Conn_01x10_Female, J2 Term_2, J3 Term_2, J4 Term_2, J6 Term_2, J7 Term_2, J8 Term_2, J9 Term_2, K2 G5Q-1, U1 MCP6001U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

Commit message: added historical scripts and new revisions
Connections:
- net /CLK renamed /TC_CLK
- net /DATA renamed /TC_DATA
- net /I2C_CLK renamed /I2C_TC_CLK
Changed lines of the file:
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@@
   (net 8 "/TMSTR1")
   (net 9 "/TMSTR2")
-  (net 10 "/I2C_CLK")
+  (net 10 "/I2C_TC_CLK")
   (net 11 "unconnected-(A1-Pad21)")
   (net 12 "/I2C_DAT")
@@
   (net 24 "/INT")
   (net 25 "/PWM")
-  (net 26 "/DATA")
-  (net 27 "/CLK")
+  (net 26 "/TC_DATA")
+  (net 27 "/TC_CLK")
   (net 28 "/SS1")
   (net 29 "/SS2")
@@
       (net 29 "/SS2") (pinfunction "D11") (pintype "bidirectional"))
     (pad "15" thru_hole oval locked (at 0 35.56) (size 1.6 1.6) (drill 1) (layers "*.Cu" "*.Mask")
-      (net 26 "/DATA") (pinfunction "D12") (pintype "bidirectional"))
+      (net 26 "/TC_DATA") (pinfunction "D12") (pintype "bidirectional"))
     (pad "16" thru_hole oval locked (at 15.24 35.56) (size 1.6 1.6) (drill 1) (layers "*.Cu" "*.Mask")
-      (net 27 "/CLK") (pinfunction "D13") (pintype "bidirectional"))
+      (net 27 "/TC_CLK") (pinfunction "D13") (pintype "bidirectional"))
     (pad "17" thru_hole oval locked (at 15.24 33.02) (size 1.6 1.6) (drill 1) (layers "*.Cu" "*.Mask")
       (net 2 "unconnected-(A1-Pad17)") (pinfunction "3V3") (pintype "power_out+no_connect"))
@@
       (net 12 "/I2C_DAT") (pinfunction "A4") (pintype "bidirectional"))
     (pad "24" thru_hole oval locked (at 15.24 15.24) (size 1.6 1.6) (drill 1) (layers "*.Cu" "*.Mask")
-      (net 10 "/I2C_CLK") (pinfunction "A5") (pintype "bidirectional"))
+      (net 10 "/I2C_TC_CLK") (pinfunction "A5") (pintype "bidirectional"))
     (pad "25" thru_hole oval locked (at 15.24 12.7) (size 1.6 1.6) (drill 1) (layers "*.Cu" "*.Mask")
       (net 17 "unconnected-(A1-Pad25)") (pinfunction "A6") (pintype "bidirectional+no_connect"))
@@
       (net 23 "+12V") (pinfunction "Pin_2") (pintype "passive"))
     (pad "3" thru_hole oval locked (at 0 5.08) (size 1.7 1.7) (drill 1) (layers "*.Cu" "*.Mask")
-      (net 10 "/I2C_CLK") (pinfunction "Pin_3") (pintype "passive"))
+      (net 10 "/I2C_TC_CLK") (pinfunction "Pin_3") (pintype "passive"))
     (pad "4" thru_hole oval locked (at 0 7.62) (size 1.7 1.7) (drill 1) (layers "*.Cu" "*.Mask")
       (net 12 "/I2C_DAT") (pinfunction "Pin_4") (pintype "passive"))
@@
   (footprint "TerminalBlock_Phoenix:TerminalBlock_Phoenix_MKDS-1,5-2_1x02_P5.00mm_Horizontal" (layer "F.Cu")
     (at 186.273 118.043 90)
-    (descr "Terminal Block Phoenix MKDS-1,5-2, 2 pins, pitch 5mm, size 10x9.8mm^2, drill diamater 1.3mm, pad diameter 2.6mm, see http://www.farnell.com/datasheets/100425.pdf, script-generated using https://github.com/pointhi/kicad-footprint-generator/scripts/TerminalBlock_Phoenix")
+    (descr "Terminal Block Phoenix MKDS-1,5-2, 2 pins, pitch 5mm, size 10x9.8mm^2, drill diamater 1.3mm, pad diameter 2.6mm, see http://www.farnell.com/TC_DATAsheets/100425.pdf, script-generated using https://github.com/pointhi/kicad-footprint-generator/scripts/TerminalBlock_Phoenix")
     (tags "THT Terminal Block Phoenix MKDS-1,5-2 pitch 5mm size 10x9.8mm^2 drill 1.3mm pad 2.6mm")
     (property "Part #" "1935161")
@@
   (footprint "TerminalBlock_Phoenix:TerminalBlock_Phoenix_MKDS-1,5-2_1x02_P5.00mm_Horizontal" (layer "F.Cu")
     (at 186.273 128.457 90)
-    (descr "Terminal Block Phoenix MKDS-1,5-2, 2 pins, pitch 5mm, size 10x9.8mm^2, drill diamater 1.3mm, pad diameter 2.6mm, see http://www.farnell.com/datasheets/100425.pdf, script-generated using https://github.com/pointhi/kicad-footprint-generator/scripts/TerminalBlock_Phoenix")
+    (descr "Terminal Block Phoenix MKDS-1,5-2, 2 pins, pitch 5mm, size 10x9.8mm^2, drill diamater 1.3mm, pad diameter 2.6mm, see http://www.farnell.com/TC_DATAsheets/100425.pdf, script-generated using https://github.com/pointhi/kicad-footprint-generator/scripts/TerminalBlock_Phoenix")
     (tags "THT Terminal Block Phoenix MKDS-1,5-2 pitch 5mm size 10x9.8mm^2 drill 1.3mm pad 2.6mm")
     (property "Part #" "1935161")
@@
   (footprint "TerminalBlock_Phoenix:TerminalBlock_Phoenix_MKDS-1,5-2_1x02_P5.00mm_Horizontal" (layer "F.Cu")
     (at 186.273 107.669 90)
-    (descr "Terminal Block Phoenix MKDS-1,5-2, 2 pins, pitch 5mm, size 10x9.8mm^2, drill diamater 1.3mm, pad diameter 2.6mm, see http://www.farnell.com/datasheets/100425.pdf, script-generated using https://github.com/pointhi/kicad-footprint-generator/scripts/TerminalBlock_Phoenix")
+    (descr "Terminal Block Phoenix MKDS-1,5-2, 2 pins, pitch 5mm, size 10x9.8mm^2, drill diamater 1.3mm, pad diameter 2.6mm, see http://www.farnell.com/TC_DATAsheets/100425.pdf, script-generated using https://github.com/pointhi/kicad-footprint-generator/scripts/TerminalBlock_Phoenix")
     (tags "THT Terminal Block Phoenix MKDS-1,5-2 pitch 5mm size 10x9.8mm^2 drill 1.3mm pad 2.6mm")
     (property "Part #" "1935161")
@@
   (footprint "TerminalBlock_Phoenix:TerminalBlock_Phoenix_MKDS-1,5-2_1x02_P5.00mm_Horizontal" (layer "F.Cu")
     (at 186.05 60.25 90)
-    (descr "Terminal Block Phoenix MKDS-1,5-2, 2 pins, pitch 5mm, size 10x9.8mm^2, drill diamater 1.3mm, pad diameter 2.6mm, see http://www.farnell.com/datasheets/100425.pdf, script-generated using https://github.com/pointhi/kicad-footprint-generator/scripts/TerminalBlock_Phoenix")
+    (descr "Terminal Block Phoenix MKDS-1,5-2, 2 pins, pitch 5mm, size 10x9.8mm^2, drill diamater 1.3mm, pad diameter 2.6mm, see http://www.farnell.com/TC_DATAsheets/100425.pdf, script-generated using https://github.com/pointhi/kicad-footprint-generator/scripts/TerminalBlock_Phoenix")
     (tags "THT Terminal Block Phoenix MKDS-1,5-2 pitch 5mm size 10x9.8mm^2 drill 1.3mm pad 2.6mm")
     (property "Part #" "1935161")
@@
   (footprint "TerminalBlock_Phoenix:TerminalBlock_Phoenix_MKDS-1,5-2_1x02_P5.00mm_Horizontal" (layer "F.Cu")
     (at 186.273 97.342 90)
-    (descr "Terminal Block Phoenix MKDS-1,5-2, 2 pins, pitch 5mm, size 10x9.8mm^2, drill diamater 1.3mm, pad diameter 2.6mm, see http://www.farnell.com/datasheets/100425.pdf, script-generated using https://github.com/pointhi/kicad-footprint-generator/scripts/TerminalBlock_Phoenix")
+    (descr "Terminal Block Phoenix MKDS-1,5-2, 2 pins, pitch 5mm, size 10x9.8mm^2, drill diamater 1.3mm, pad diameter 2.6mm, see http://www.farnell.com/TC_DATAsheets/100425.pdf, script-generated using https://github.com/pointhi/kicad-footprint-generator/scripts/TerminalBlock_Phoenix")
     (tags "THT Terminal Block Phoenix MKDS-1,5-2 pitch 5mm size 10x9.8mm^2 drill 1.3mm pad 2.6mm")
     (property "Part #" "1935161")
@@
   (footprint "TerminalBlock_Phoenix:TerminalBlock_Phoenix_MKDS-1,5-2_1x02_P5.00mm_Horizontal" (layer "F.Cu")
     (at 186.05 81.4 90)
-    (descr "Terminal Block Phoenix MKDS-1,5-2, 2 pins, pitch 5mm, size 10x9.8mm^2, drill diamater 1.3mm, pad diameter 2.6mm, see http://www.farnell.com/datasheets/100425.pdf, script-generated using https://github.com/pointhi/kicad-footprint-generator/scripts/TerminalBlock_Phoenix")
+    (descr "Terminal Block Phoenix MKDS-1,5-2, 2 pins, pitch 5mm, size 10x9.8mm^2, drill diamater 1.3mm, pad diameter 2.6mm, see http://www.farnell.com/TC_DATAsheets/100425.pdf, script-generated using https://github.com/pointhi/kicad-footprint-generator/scripts/TerminalBlock_Phoenix")
     (tags "THT Terminal Block Phoenix MKDS-1,5-2 pitch 5mm size 10x9.8mm^2 drill 1.3mm pad 2.6mm")
     (property "Part #" "1935161")
@@
   (footprint "TerminalBlock_Phoenix:TerminalBlock_Phoenix_MKDS-1,5-2_1x02_P5.00mm_Horizontal" (layer "F.Cu")
     (at 186.054 70.799 90)
-    (descr "Terminal Block Phoenix MKDS-1,5-2, 2 pins, pitch 5mm, size 10x9.8mm^2, drill diamater 1.3mm, pad diameter 2.6mm, see http://www.farnell.com/datasheets/100425.pdf, script-generated using https://github.com/pointhi/kicad-footprint-generator/scripts/TerminalBlock_Phoenix")
+    (descr "Terminal Block Phoenix MKDS-1,5-2, 2 pins, pitch 5mm, size 10x9.8mm^2, drill diamater 1.3mm, pad diameter 2.6mm, see http://www.farnell.com/TC_DATAsheets/100425.pdf, script-generated using https://github.com/pointhi/kicad-footprint-generator/scripts/TerminalBlock_Phoenix")
     (tags "THT Terminal Block Phoenix MKDS-1,5-2 pitch 5mm size 10x9.8mm^2 drill 1.3mm pad 2.6mm")
     (property "Part #" "1935161")
@@
       (net 5 "+5V") (pinfunction "VCC") (pintype "power_in"))
     (pad "5" smd roundrect (at 2.475 -1.905 180) (size 1.97 0.59) (layers "B.Cu" "B.Paste" "B.Mask") (roundrect_rratio 0.07)
-      (net 27 "/CLK") (pinfunction "SCK") (pintype "input"))
+      (net 27 "/TC_CLK") (pinfunction "SCK") (pintype "input"))
     (pad "6" smd roundrect (at 2.475 -0.635 180) (size 1.97 0.59) (layers "B.Cu" "B.Paste" "B.Mask") (roundrect_rratio 0.07)
       (net 29 "/SS2") (pinfunction "~{CS}") (pintype "input"))
     (pad "7" smd roundrect (at 2.475 0.635 180) (size 1.97 0.59) (layers "B.Cu" "B.Paste" "B.Mask") (roundrect_rratio 0.07)
-      (net 26 "/DATA") (pinfunction "SO") (pintype "output"))
+      (net 26 "/TC_DATA") (pinfunction "SO") (pintype "output"))
     (pad "8" smd roundrect (at 2.475 1.905 180) (size 1.97 0.59) (layers "B.Cu" "B.Paste" "B.Mask") (roundrect_rratio 0.07)
       (net 36 "unconnected-(U4-Pad8)") (pinfunction "N.C.") (pintype "bidirectional+no_connect"))
@@
       (net 5 "+5V") (pinfunction "VCC") (pintype "power_in"))
     (pad "5" smd roundrect (at 2.475 -1.905 180) (size 1.97 0.59) (layers "B.Cu" "B.Paste" "B.Mask") (roundrect_rratio 0.07)
-      (net 27 "/CLK") (pinfunction "SCK") (pintype "input"))
+      (net 27 "/TC_CLK") (pinfunction "SCK") (pintype "input"))
     (pad "6" smd roundrect (at 2.475 -0.635 180) (size 1.97 0.59) (layers "B.Cu" "B.Paste" "B.Mask") (roundrect_rratio 0.07)
       (net 28 "/SS1") (pinfunction "~{CS}") (pintype "input"))
     (pad "7" smd roundrect (at 2.475 0.635 180) (size 1.97 0.59) (layers "B.Cu" "B.Paste" "B.Mask") (roundrect_rratio 0.07)
-      (net 26 "/DATA") (pinfunction "SO") (pintype "output"))
+      (net 26 "/TC_DATA") (pinfunction "SO") (pintype "output"))
     (pad "8" smd roundrect (at 2.475 1.905 180) (size 1.97 0.59) (layers "B.Cu" "B.Paste" "B.Mask") (roundrect_rratio 0.07)
       (net 33 "unconnected-(U3-Pad8)") (pinfunction "N.C.") (pintype "bidirectional+no_connect"))
