File: hardware/BREAD_Slice.kicad_pcb (KiCad board)
At the start: 2 copper layers, 70 x 100 mm, 41 parts, among them J1 Conn_01x10_Female, J2 Screw_Terminal_01x02, J3 Screw_Terminal_01x02, J4 Screw_Terminal_01x06, J5 Screw_Terminal_01x06, K1 G5Q-1, K2 G5Q-1, U2 MAX31855KASA, U3 MAX31855KASA, U4 TCMT1100, U5 TCMT1100

Commit message: feat: update to kicad 10 and migrate old references to kml
Parts:
- HS1: footprint KMLib_Mounting:Thermal Pad -> KMLib_Mounting:Thermal_Pad
