File: hardware/BREAD_Slice.kicad_sch (KiCad schematic)
At the start: 22 parts, among them J1 Conn_01x10_Female, J2 Screw_Terminal_01x02, J3 Screw_Terminal_01x02, J4 Screw_Terminal_01x06, J5 Screw_Terminal_01x06, SW1 ESTOP, SW2 ESTOP

Commit message: feat: update to kicad 10 and migrate old references to kml
Parts:
- HS1: footprint KMLib_Mounting:Thermal Pad -> KMLib_Mounting:Thermal_Pad
- U1: value ~ -> (none)
